File: PicoDrive.kicad_pcb (KiCad board)
At the start: 2 copper layers, 31.8 x 20.3 mm, 55 parts, among them J1 M1, J2 M2, J3 M3, J4 RECEIVER, P1 USB_C_Plug_USB2.0, U1 W25Q32JVSS, U2 XC6206PxxxMR, U3 RP2040, U4 DRV8837, U5 DRV8837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

Commit message: As ordered
Parts:
- J1, J2, J3: footprint Connector_JST:JST_SH_BM02B-SRSS-TB_1x02-1MP_P1.00mm_Vertical -> Connector_JST:JST_SH_SM02B-SRSS-TB_1x02-1MP_P1.00mm_Horizontal
- J4: footprint Connector_JST:JST_SH_BM03B-SRSS-TB_1x03-1MP_P1.00mm_Vertical -> Connector_JST:JST_SH_SM03B-SRSS-TB_1x03-1MP_P1.00mm_Horizontal
- moved C17 4.57 mm to (161.9, 69.2), turned to -90 degrees
- moved C20 4.22 mm to (164.4, 70.2), turned to 180 degrees
- moved C19 2.16 mm to (166.6, 66.9)
- moved U5 1.91 mm to (164.5, 65.4)
- moved U6 1.91 mm to (164.5, 68.3)
- moved C18 1.65 mm to (167.1, 64.1), turned to 180 degrees
- moved C16 1.30 mm to (161.9, 65.7), turned to 90 degrees
- moved R12 1.20 mm to (167.5, 52.7), turned to -90 degrees
- moved C6 0.99 mm to (166.5, 54.6), turned to 90 degrees
- moved C5 0.76 mm to (164.1, 59.9)
- moved U4 0.76 mm to (165.6, 62.2)
- moved C15 0.63 mm to (162.9, 63.5)
- moved C13 0.38 mm to (161.9, 61.7)
- moved C1 0.38 mm to (149.6, 66.5)
- moved Y1 0.38 mm to (166.6, 57.8)
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- renumbered C5 to C2, C2 to C3, C6 to C4, C3 to C5, C4 to C6
Connections:
- J1 pad 1: /M1- -> /M1+
- J1 pad 2: /M1+ -> /M1-
- J2 pad 1: /M2- -> /M2+
- J2 pad 2: /M2+ -> /M2-
- J3 pad 1: /M3- -> /M3+
- J3 pad 2: /M3+ -> /M3-
- J4 pad 1: +3V3 -> /IBUS
- J4 pad 3: /IBUS -> +3V3
Routing:
- net +BATT: track 45.6 -> 43.3 mm
- net /M2B: track 8.71 -> 6.80 mm
- net /M2A: track 9.41 -> 7.51 mm
- net +3V3: track 95.7 -> 93.9 mm
- net /M3B: track 11.7 -> 10.1 mm
- net /M3A: track 12.4 -> 10.8 mm
- net GND: track 32.7 -> 31.2 mm, vias 39 -> 41
- net /M3+: track 3.58 -> 4.87 mm
- net Net-(C5-Pad1): track 7.94 -> 6.74 mm
- net /M3-: track 3.50 -> 4.68 mm
- net /M2-: track 6.83 -> 7.84 mm
- net /M2+: track 6.75 -> 7.63 mm
- net /M1A: track 7.75 -> 6.96 mm
- net /M1B: track 7.10 -> 6.34 mm
- net (no net): vias 0 -> 2
Other:
- board size 31.8 x 20.3 mm -> 32.8 x 20.3 mm
