File: PicoDrive.kicad_sch (KiCad schematic)
At the start: 55 parts, among them J1 M1, J2 M2, J3 M3, J4 RECEIVER, P1 USB_C_Plug_USB2.0, U1 W25Q32JVSS, U2 XC6206PxxxMR, U3 RP2040, U4 DRV8837, U5 DRV8837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

Commit message: As ordered
Parts:
- J1, J2, J3: footprint Connector_JST:JST_SH_BM02B-SRSS-TB_1x02-1MP_P1.00mm_Vertical -> Connector_JST:JST_SH_SM02B-SRSS-TB_1x02-1MP_P1.00mm_Horizontal
- J4: footprint Connector_JST:JST_SH_BM03B-SRSS-TB_1x03-1MP_P1.00mm_Vertical -> Connector_JST:JST_SH_SM03B-SRSS-TB_1x03-1MP_P1.00mm_Horizontal
- renumbered C5 to C2, C2 to C3, C6 to C4, C3 to C5, C4 to C6
Connections:
- net +3V3: now also J4.3 (Pin_3); no longer J4.1 (Pin_1)
- net IBUS: now also J4.1 (Pin_1); no longer J4.3 (Pin_3)
- net M1+: now also J1.1 (Pin_1); no longer J1.2 (Pin_2)
- net M1-: now also J1.2 (Pin_2); no longer J1.1 (Pin_1)
- net M2+: now also J2.1 (Pin_1); no longer J2.2 (Pin_2)
- net M2-: now also J2.2 (Pin_2); no longer J2.1 (Pin_1)
- net M3+: now also J3.1 (Pin_1); no longer J3.2 (Pin_2)
- net M3-: now also J3.2 (Pin_2); no longer J3.1 (Pin_1)
