File: hardware/PicoDrive.kicad_pcb (KiCad board)
At the start: 2 copper layers, 32.8 x 20.3 mm, 55 parts, among them J1 M1, J2 M2, J3 M3, J4 RECEIVER, P1 USB_C_Plug_USB2.0, U1 W25Q32JVSS, U2 XC6206PxxxMR, U3 RP2040, U4 DRV8837, U5 DRV8837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

Commit message: Started firmware
Also fixed an error on the PCB layout
Routing:
- net GND: vias 41 -> 43
- net (no net): vias 2 -> 0
Changed lines of the file:
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@@
     (style (thickness 0.2) (arrow_length 1.27) (text_position_mode 0) (extension_height 0.58642) (extension_offset 0.5) keep_text_aligned)
   )
-  (via (at 142.875 63.5) (size 0.5) (drill 0.3) (layers "F.Cu" "B.Cu") (free) (net 0))
-  (via (at 146.685 64.77) (size 0.5) (drill 0.3) (layers "F.Cu" "B.Cu") (free) (net 0))
   (segment (start 152.4 62.286172) (end 151.734523 61.620695) (width 0.5) (layer "F.Cu") (net 1))
   (segment (start 156.972 59.182) (end 156.972 56.896) (width 0.3) (layer "F.Cu") (net 1))
@@
   (via (at 167.64 71.12) (size 0.5) (drill 0.3) (layers "F.Cu" "B.Cu") (free) (net 3))
   (via (at 150.876 53.34) (size 0.5) (drill 0.3) (layers "F.Cu" "B.Cu") (free) (net 3))
+  (via (at 142.875 63.5) (size 0.5) (drill 0.3) (layers "F.Cu" "B.Cu") (free) (net 3))
   (via (at 170.18 71.12) (size 0.5) (drill 0.3) (layers "F.Cu" "B.Cu") (free) (net 3))
   (via (at 161.163 67.945) (size 0.5) (drill 0.3) (layers "F.Cu" "B.Cu") (free) (net 3))
@@
   (via (at 157.099 65.151) (size 0.5) (drill 0.3) (layers "F.Cu" "B.Cu") (free) (net 3))
   (via (at 165.1 53.34) (size 0.5) (drill 0.3) (layers "F.Cu" "B.Cu") (free) (net 3))
+  (via (at 146.685 64.77) (size 0.5) (drill 0.3) (layers "F.Cu" "B.Cu") (free) (net 3))
   (via (at 162.56 52.07) (size 0.5) (drill 0.3) (layers "F.Cu" "B.Cu") (free) (net 3))
   (via (at 164.465 71.12) (size 0.5) (drill 0.3) (layers "F.Cu" "B.Cu") (free) (net 3))
